Commit message: 8/16

File: catkin_ws/src/my_robot/urdf/my_robot.xacro (robot description, xacro)
@@ -149,5 +149,5 @@
     <link name='hokuyo'>
       <collision name='hokuyo_collision'>
-        <origin xyz = '0 0 0' rpy = '0 0 0'/>
+        <origin xyz = '-1 0 0' rpy = '0 0 0'/>
         <geometry>
           <box size = '0.1 0.1 0.1'/>
@@ -155,5 +155,5 @@
       </collision>
       <visual name='hokuyo_visual'>
-        <origin xyz = '0 0 0' rpy = '0 0 0'/>
+        <origin xyz = '-1 0 0' rpy = '0 0 0'/>
         <geometry>
           <mesh filename = "package://my_robot/meshes/hokuyo.dae"/>
